File: DDR4-SODIMM/ddr4-sodimm/ddr4-sodimm.kicad_pcb (KiCad board)
At the start: 2 copper layers, 69.6 x 30 mm, 1 part

Commit message: add DDR4 SODIMM board informations
Other:
- copper layers 2 -> 6
Changed lines of the file:
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@@
 (kicad_pcb (version 20221018) (generator pcbnew)
   (general
-    (thickness 1.6)
+    (thickness 1.2)
   )
   (paper "A4")
   (layers
     (0 "F.Cu" signal)
+    (1 "In1.Cu" signal)
+    (2 "In2.Cu" signal)
+    (3 "In3.Cu" signal)
+    (4 "In4.Cu" signal)
     (31 "B.Cu" signal)
     (32 "B.Adhes" user "B.Adhesive")
@@
   )
   (setup
+    (stackup
+      (layer "F.SilkS" (type "Top Silk Screen"))
+      (layer "F.Paste" (type "Top Solder Paste"))
+      (layer "F.Mask" (type "Top Solder Mask") (thickness 0.01))
+      (layer "F.Cu" (type "copper") (thickness 0.035))
+      (layer "dielectric 1" (type "prepreg") (thickness 0.1) (material "3313") (epsilon_r 4.5) (loss_tangent 0.02))
+      (layer "In1.Cu" (type "copper") (thickness 0.0152))
+      (layer "dielectric 2" (type "core") (thickness 0.3746) (material "FR4") (epsilon_r 4.5) (loss_tangent 0.02))
+      (layer "In2.Cu" (type "copper") (thickness 0.0152))
+      (layer "dielectric 3" (type "prepreg") (thickness 0.1) (material "2116") (epsilon_r 4.5) (loss_tangent 0.02))
+      (layer "In3.Cu" (type "copper") (thickness 0.0152))
+      (layer "dielectric 4" (type "core") (thickness 0.3746) (material "FR4") (epsilon_r 4.5) (loss_tangent 0.02))
+      (layer "In4.Cu" (type "copper") (thickness 0.0152))
+      (layer "dielectric 5" (type "prepreg") (thickness 0.1) (material "3313") (epsilon_r 4.5) (loss_tangent 0.02))
+      (layer "B.Cu" (type "copper") (thickness 0.035))
+      (layer "B.Mask" (type "Bottom Solder Mask") (thickness 0.01))
+      (layer "B.Paste" (type "Bottom Solder Paste"))
+      (layer "B.SilkS" (type "Bottom Silk Screen"))
+      (copper_finish "None")
+      (dielectric_constraints yes)
+    )
     (pad_to_mask_clearance 0)
-    (aux_axis_origin 100.2 99.5)
+    (aux_axis_origin 100 100)
     (pcbplotparams
       (layerselection 0x00010fc_ffffffff)
